File: hardware/badge/Revision A2/oshcamp23-badge-RevA2.brd (EAGLE design)
At the start: 75 x 120 mm, 58 parts, among them CON2 STEMMA_I2C_QT, IC2 LD1117-3.3, IC3 WMCU-ESP8285H16, J1 61030621121, P1 Buzzer, Q1 SS8050, Q2 SS8050, Q3 SS8050

Commit message: add iboms for both kit variants
Parts:
- CON1: value (none) -> USBC_C-31-M-12
- IC1: value (none) -> CH343G
- L1: value TBD -> 0R LINK (Temp)
- SW1, SW2, SW3, SW4, SW5, SW6, SW7: value (none) -> Pushbutton
